File: hardware/HW-LEEK-001/HW-LEEK-001.kicad_pcb (KiCad board)
At the start: 2 copper layers, 73.2 x 96.2 mm, 24 parts, among them J1 Conn_01x03_Pin, U1 ATtiny402-SS

Commit message: HW Revision 02
Parts:
- D4, D5, D6, D7: footprint LED_SMD:LED_0603_1608Metric -> LED_SMD:LED_0805_2012Metric
- moved R2 3.07 mm to (169.0, 70.9), turned to 0 degrees
- moved R3 1.89 mm to (144.8, 95.0)
- turned D1 to 180 degrees
Connections:
- D1 pad 2: /GREEN_LED -> /GREEN_GROUP_2
- D2 pad 2: /GREEN_LED -> /GREEN_GROUP_2
- D3 pad 2: /GREEN_LED -> /GREEN_GROUP_2
- D4 pad 2: /GREEN_LED -> /GREEN_GROUP_1
- D5 pad 2: /GREEN_LED -> /GREEN_GROUP_1
- D6 pad 2: /WHITE_LED -> /WHITE_GROUP_1
- D7 pad 2: /WHITE_LED -> /WHITE_GROUP_2
- SW3 pad 1: /BATT+ -> unconnected-(SW3-Pad1)
- SW3 pad 2: unconnected-(SW3-Pad2) -> /BATT+
- U1 pad 2: /GREEN_LED -> /GREEN_GROUP_2
- U1 pad 3: /WHITE_LED -> /WHITE_GROUP_2
- U1 pad 4: /UPDI -> /GREEN_GROUP_1
- U1 pad 6: unconnected-(U1-~{RESET}/PA0-Pad6) -> /UPDI
- U1 pad 7: unconnected-(U1-PA3-Pad7) -> /WHITE_GROUP_1
Routing:
- net /GREEN_LED: track 75.8 -> 0.00 mm, vias 5 -> 0
- net /GREEN_GROUP_1: track 0.00 -> 60.7 mm, vias 0 -> 2
- net /WHITE_LED: track 58.1 -> 0.00 mm, vias 2 -> 0
- net /WHITE_GROUP_2: track 0.00 -> 53.8 mm, vias 0 -> 3
- net /GREEN_GROUP_2: track 0.00 -> 40.6 mm, vias 0 -> 3
- net /WHITE_GROUP_1: track 0.00 -> 37.1 mm, vias 0 -> 3
- net +3V0: track 78.2 -> 89.9 mm
- net /BATT+: track 77.5 -> 74.9 mm
- net /UPDI: track 63.4 -> 64.4 mm
- net GND: track 10.1 -> 9.45 mm
Other:
- board text added: "CR1220"
- board text added: "Change Pattern 切换动画"
- board text added: "Power 开关"
- board text added: "UPDI->"

Commit message: Update final hardware
Parts:
- BT1: footprint footprints:BAT-SMD_MY-1220-03 -> EasyEDA_Lib:BAT-SMD_CR1220-2ZX
- moved G*** 6.23 mm to (139.4, 107.3)
Routing:
- net /BATT+: track 74.9 -> 68.6 mm
- net /UPDI: track 64.4 -> 66.2 mm
- net /WHITE_GROUP_2: track 53.8 -> 52.5 mm
- net GND: track 9.45 -> 8.54 mm, vias 4 -> 2
