File: hardware/HW-LEEK-001/HW-LEEK-001.kicad_sch (KiCad schematic)
At the start: 20 parts, among them J1 Conn_01x03_Pin, U1 ATtiny402-SS

Commit message: HW Revision 02
Parts:
- D4, D5, D6, D7: footprint LED_SMD:LED_0603_1608Metric -> LED_SMD:LED_0805_2012Metric
Connections:
- net BATT+: now also SW3.2; no longer SW3.1
- net UPDI: now also U1.6 (~{RESET}/PA0); no longer U1.4 (PA1)
- net WHITE_GROUP_1: now reaches U1.7 (PA3)
- net WHITE_GROUP_1: now also D6.2 (A)
- net GREEN_LED renamed GREEN_GROUP_2
- net GREEN_GROUP_2: no longer D4.2 (A), D5.2 (A)
- net WHITE_LED renamed WHITE_GROUP_2
- net WHITE_GROUP_2: no longer D6.2 (A)
- new net GREEN_GROUP_1: D4.2 (A), D5.2 (A), U1.4 (PA1)
- no-connect marks 7 -> 5
Changed lines of the file:
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@@
 		(title "HW-LEEK-001")
 		(date "2026-03-09")
-		(rev "1")
+		(rev "2")
 		(company "Diva Engineering")
 	)
@@
 	)
 	(junction
-		(at 219.71 91.44)
-		(diameter 0)
-		(color 0 0 0 0)
-	)
-	(junction
 		(at 154.94 114.3)
 		(diameter 0)
@@
 	)
 	(no_connect
-		(at 120.65 85.09)
+		(at 125.73 85.09)
 	)
 	(no_connect
@@
 	)
 	(no_connect
-		(at 106.68 96.52)
-	)
-	(no_connect
-		(at 106.68 104.14)
-	)
-	(no_connect
 		(at 105.41 85.09)
 	)
@@
 	(wire
 		(pts
-			(xy 219.71 104.14) (xy 219.71 91.44)
-		)
-		(stroke
-			(width 0)
-			(type default)
-		)
-	)
-	(wire
-		(pts
 			(xy 156.21 91.44) (xy 154.94 91.44)
 		)
@@
 	(wire
 		(pts
-			(xy 198.12 80.01) (xy 198.12 91.44)
-		)
-		(stroke
-			(width 0)
-			(type default)
-		)
-	)
-	(wire
-		(pts
-			(xy 106.68 99.06) (xy 119.38 99.06)
+			(xy 198.12 73.66) (xy 198.12 91.44)
+		)
+		(stroke
+			(width 0)
+			(type default)
+		)
+	)
+	(wire
+		(pts
+			(xy 106.68 96.52) (xy 123.19 96.52)
 		)
 		(stroke
@@
 	(wire
 		(pts
-			(xy 106.68 106.68) (xy 119.38 106.68)
+			(xy 106.68 106.68) (xy 123.19 106.68)
 		)
 		(stroke
@@
 	(wire
 		(pts
-			(xy 219.71 80.01) (xy 219.71 91.44)
+			(xy 219.71 73.66) (xy 219.71 91.44)
 		)
 		(stroke
@@
 	(wire
 		(pts
+			(xy 106.68 104.14) (xy 123.19 104.14)
+		)
+		(stroke
+			(width 0)
+			(type default)
+		)
+	)
+	(wire
+		(pts
 			(xy 143.51 29.21) (xy 128.27 29.21)
 		)
@@
 	(wire
 		(pts
+			(xy 120.65 85.09) (xy 120.65 87.63)
+		)
+		(stroke
+			(width 0)
+			(type default)
+		)
+	)
+	(wire
+		(pts
 			(xy 26.67 46.99) (xy 35.56 46.99)
 		)
@@
 	(wire
 		(pts
-			(xy 125.73 86.36) (xy 135.89 86.36)
-		)
-		(stroke
-			(width 0)
-			(type default)
-		)
-	)
-	(wire
-		(pts
 			(xy 57.15 87.63) (xy 57.15 100.33)
 		)
@@
 	(wire
 		(pts
-			(xy 176.53 80.01) (xy 176.53 91.44)
+			(xy 176.53 73.66) (xy 176.53 91.44)
 		)
 		(stroke
@@
 	(wire
 		(pts
+			(xy 120.65 87.63) (xy 135.89 87.63)
+		)
+		(stroke
+			(width 0)
+			(type default)
+		)
+	)
+	(wire
+		(pts
 			(xy 128.27 39.37) (xy 128.27 41.91)
 		)
@@
 	(wire
 		(pts
-			(xy 106.68 109.22) (xy 119.38 109.22)
+			(xy 106.68 109.22) (xy 123.19 109.22)
 		)
 		(stroke
@@
 	(wire
 		(pts
+			(xy 106.68 99.06) (xy 123.19 99.06)
+		)
+		(stroke
+			(width 0)
+			(type default)
+		)
+	)
+	(wire
+		(pts
 			(xy 140.97 31.75) (xy 143.51 31.75)
 		)
@@
 	(wire
 		(pts
-			(xy 125.73 85.09) (xy 125.73 86.36)
-		)
-		(stroke
-			(width 0)
-			(type default)
-		)
-	)
-	(wire
-		(pts
 			(xy 199.39 104.14) (xy 200.66 104.14)
 		)
@@
 	(wire
 		(pts
-			(xy 106.68 101.6) (xy 119.38 101.6)
+			(xy 106.68 101.6) (xy 123.19 101.6)
+		)
+		(stroke
+			(width 0)
+			(type default)
+		)
+	)
+	(wire
+		(pts
+			(xy 219.71 104.14) (xy 219.71 121.92)
 		)
 		(stroke
@@
 		)
 	)
-	(label "WHITE_LED"
-		(at 119.38 109.22 180)
+	(label "WHITE_GROUP_1"
+		(at 219.71 73.66 270)
 		(effects
 			(font
@@
 		)
 	)
-	(label "GREEN_LED"
-		(at 198.12 80.01 270)
+	(label "BATT+"
+		(at 135.89 87.63 180)
 		(effects
 			(font
@@
 		)
 	)
-	(label "GREEN_LED"
-		(at 176.53 80.01 270)
+	(label "GREEN_GROUP_2"
+		(at 123.19 106.68 180)
 		(effects
 			(font
@@
 		)
 	)
-	(label "BATT+"
-		(at 135.89 86.36 180)
+	(label "GREEN_GROUP_2"
+		(at 198.12 73.66 270)
 		(effects
 			(font
@@
 	)
 	(label "SELECT"
-		(at 119.38 101.6 180)
+		(at 123.19 101.6 180)
+		(effects
+			(font
+				(size 1.27 1.27)
+			)
+			(justify right bottom)
+		)
+	)
+	(label "WHITE_GROUP_2"
+		(at 219.71 121.92 90)
+		(effects
+			(font
+				(size 1.27 1.27)
+			)
+			(justify left bottom)
+		)
+	)
+	(label "GREEN_GROUP_1"
+		(at 176.53 73.66 270)
 		(effects
 			(font
@@
 		)
 	)
+	(label "WHITE_GROUP_2"
+		(at 123.19 109.22 180)
+		(effects
+			(font
+				(size 1.27 1.27)
+			)
+			(justify right bottom)
+		)
+	)
 	(label "SELECT"
 		(at 118.11 31.75 0)
@@
 		)
 	)
+	(label "GREEN_GROUP_1"
+		(at 123.19 99.06 180)
+		(effects
+			(font
+				(size 1.27 1.27)
+			)
+			(justify right bottom)
+		)
+	)
 	(label "BATT+"
 		(at 25.4 34.29 0)
@@
 		)
 	)
-	(label "GREEN_LED"
-		(at 119.38 106.68 180)
+	(label "UPDI"
+		(at 123.19 96.52 180)
 		(effects
 			(font
@@
 		)
 	)
-	(label "UPDI"
-		(at 119.38 99.06 180)
-		(effects
-			(font
-				(size 1.27 1.27)
-			)
-			(justify right bottom)
-		)
-	)
-	(label "WHITE_LED"
-		(at 219.71 80.01 270)
+	(label "WHITE_GROUP_1"
+		(at 123.19 104.14 180)
 		(effects
 			(font
@@
 			)
 		)
-		(property "Footprint" "LED_SMD:LED_0603_1608Metric"
+		(property "Footprint" "LED_SMD:LED_0805_2012Metric"
 			(at 170.18 104.14 0)
 			(effects
@@
 			)
 		)
-		(property "Footprint" "LED_SMD:LED_0603_1608Metric"
+		(property "Footprint" "LED_SMD:LED_0805_2012Metric"
 			(at 170.18 91.44 0)
 			(effects
@@
 			)
 		)
-		(property "Footprint" "LED_SMD:LED_0603_1608Metric"
+		(property "Footprint" "LED_SMD:LED_0805_2012Metric"
 			(at 214.63 91.44 0)
 			(effects
@@
 			)
 		)
-		(property "Footprint" "LED_SMD:LED_0603_1608Metric"
+		(property "Footprint" "LED_SMD:LED_0805_2012Metric"
 			(at 214.63 104.14 0)
 			(effects

Commit message: Update final hardware
Parts:
- BT1: footprint footprints:BAT-SMD_MY-1220-03 -> EasyEDA_Lib:BAT-SMD_CR1220-2ZX
Changed lines of the file:
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@@
 			)
 		)
-		(property "Footprint" "footprints:BAT-SMD_MY-1220-03"
+		(property "Footprint" "EasyEDA_Lib:BAT-SMD_CR1220-2ZX"
 			(at 35.56 39.116 90)
 			(effects
